Commit message: SLAM finito

File: src/rosbot_description/urdf/rosbot.xacro (robot description, xacro)
@@ -9,5 +9,5 @@
   <link name="base_link"></link>
   <joint name="base_link_joint" type="fixed">
-    <origin xyz="0 1 0" rpy="0 0 0"/>
+    <origin xyz="0 0 0" rpy="0 0 0"/>
     <parent link="base_link"/>
     <child link="body_link"/>
